Commit message: Four_wheels added

File: description/gazebo_control.xacro (robot description, xacro)
@@ -4,6 +4,8 @@
         <plugin name="diff_drive" filename="libgazebo_ros_diff_drive.so">
             <!-- Wheel Information -->
-            <left_joint>left_wheel_joint</left_joint>
-            <right_joint>right_wheel_joint</right_joint>
+            <left_rear_joint>left_rear_wheel_joint</left_rear_joint>
+            <left_joint>left_front_wheel_joint</left_joint>
+            <right_rear_joint>right_rear_wheel_joint</right_rear_joint>
+            <right_joint>right_front_wheel_joint</right_joint>
             <wheel_separation>0.35</wheel_separation>
             <wheel_diameter>0.1</wheel_diameter>

File: description/robot_core.xacro (robot description, xacro)
@@ -26,18 +26,18 @@
     <link name="chassis">
         <visual>
-            <origin xyz="0.15 0 0.075" rpy="0 0 0"/>
+            <origin xyz="0.25 0 0.075" rpy="0 0 0"/>
             <geometry>
-                <box size="0.3 0.3 0.15"/>
+                <box size="0.5 0.3 0.15"/>
             </geometry>
             <material name="white"/>
         </visual>
         <collision>
-            <origin xyz="0.15 0 0.075" rpy="0 0 0"/>
+            <origin xyz="0.25 0 0.075" rpy="0 0 0"/>
             <geometry>
-                <box size="0.3 0.3 0.15"/>
+                <box size="0.5 0.3 0.15"/>
             </geometry>
         </collision>
-        <xacro:inertial_box mass="0.5" x="0.3" y="0.3" z="0.15">
-            <origin xyz="0.15 0 0.075" rpy="0 0 0"/>
+        <xacro:inertial_box mass="0.5" x="0.5" y="0.3" z="0.15">
+            <origin xyz="0.25 0 0.075" rpy="0 0 0"/>
         </xacro:inertial_box>
     </link>
@@ -45,12 +45,12 @@
         <material>Gazebo/White</material>
     </gazebo>
-    <!-- LEFT WHEEL -->
-    <joint name="left_wheel_joint" type="continuous">
+    <!-- LEFT FRONT WHEEL -->
+    <joint name="left_front_wheel_joint" type="continuous">
         <parent link="base_link"/>
-        <child link="left_wheel"/>
-        <origin xyz="0 0.175 0" rpy="-${pi/2} 0 0"/>
+        <child link="left_front_wheel"/>
+        <origin xyz="0.3 0.175 0" rpy="-${pi/2} 0 0"/>
         <axis xyz="0 0 1"/>
     </joint>
-    <link name="left_wheel">
+    <link name="left_front_wheel">
         <visual>
             <geometry>
@@ -68,15 +68,15 @@
         </xacro:inertial_cylinder>
     </link>
-    <gazebo reference="left_wheel">
+    <gazebo reference="left_front_wheel">
         <material>Gazebo/Blue</material>
     </gazebo>
-    <!-- RIGHT WHEEL -->
-    <joint name="right_wheel_joint" type="continuous">
+    <!-- LEFT REAR WHEEL -->
+    <joint name="left_rear_wheel_joint" type="continuous">
         <parent link="base_link"/>
-        <child link="right_wheel"/>
-        <origin xyz="0 -0.175 0" rpy="${pi/2} 0 0"/>
-        <axis xyz="0 0 -1"/>
+        <child link="left_rear_wheel"/>
+        <origin xyz="0 0.175 0" rpy="-${pi/2} 0 0"/>
+        <axis xyz="0 0 1"/>
     </joint>
-    <link name="right_wheel">
+    <link name="left_rear_wheel">
         <visual>
             <geometry>
@@ -94,33 +94,58 @@
         </xacro:inertial_cylinder>
     </link>
-    <gazebo reference="right_wheel">
+    <gazebo reference="left_rear_wheel">
         <material>Gazebo/Blue</material>
     </gazebo>
-    <!-- CASTER WHEEL -->
-    <joint name="caster_wheel_joint" type="fixed">
-        <parent link="chassis"/>
-        <child link="caster_wheel"/>
-        <origin xyz="0.24 0 0" rpy="0 0 0"/>
+    <!-- RIGHT FRONT WHEEL -->
+    <joint name="right_front_wheel_joint" type="continuous">
+        <parent link="base_link"/>
+        <child link="right_front_wheel"/>
+        <origin xyz="0.3 -0.175 0" rpy="${pi/2} 0 0"/>
+        <axis xyz="0 0 -1"/>
     </joint>
-    <link name="caster_wheel">
+    <link name="right_front_wheel">
         <visual>
             <geometry>
-                <sphere radius="0.05" />
+                <cylinder length="0.04" radius="0.05" />
             </geometry>
-            <material name="black"/>
+            <material name="blue"/>
         </visual>
         <collision>
             <geometry>
-                <sphere radius="0.05" />
+                <cylinder length="0.04" radius="0.05" />
             </geometry>
         </collision>
-        <xacro:inertial_sphere mass="0.1" radius="0.05">
+        <xacro:inertial_cylinder mass="0.1" length="0.04" radius="0.05">
             <origin xyz="0 0 0" rpy="0 0 0"/>
-        </xacro:inertial_sphere>
+        </xacro:inertial_cylinder>
     </link>
-    <gazebo reference="caster_wheel">
-        <material>Gazebo/Black</material>
-        <mu1 value="0.001"/>
-        <mu2 value="0.001"/>
+    <gazebo reference="right_front_wheel">
+        <material>Gazebo/Blue</material>
+    </gazebo>
+    <!-- RIGHT REAR WHEEL -->
+    <joint name="right_rear_wheel_joint" type="continuous">
+        <parent link="base_link"/>
+        <child link="right_rear_wheel"/>
+        <origin xyz="0 -0.175 0" rpy="${pi/2} 0 0"/>
+        <axis xyz="0 0 -1"/>
+    </joint>
+    <link name="right_rear_wheel">
+        <visual>
+            <geometry>
+                <cylinder length="0.04" radius="0.05" />
+            </geometry>
+            <material name="blue"/>
+        </visual>
+        <collision>
+            <geometry>
+                <cylinder length="0.04" radius="0.05" />
+            </geometry>
+        </collision>
+        <xacro:inertial_cylinder mass="0.1" length="0.04" radius="0.05">
+            <origin xyz="0 0 0" rpy="0 0 0"/>
+        </xacro:inertial_cylinder>
+    </link>
+    <gazebo reference="right_rear_wheel">
+        <material>Gazebo/Blue</material>
     </gazebo>
 </robot>

Commit message: demo car implemented

File: description/gazebo_control.xacro (robot description, xacro)
@@ -6,11 +6,11 @@
             <num_wheel_pairs>2</num_wheel_pairs>
             <!-- Wheel Information -->
-            <left_joint>left_front_wheel_joint</left_joint>
-            <right_joint>right_front_wheel_joint</right_joint>
-            <left_joint>left_rear_wheel_joint</left_joint>
-            <right_joint>right_rear_wheel_joint</right_joint>
+            <left_joint>rear_left_wheel_joint</left_joint>
+            <right_joint>rear_right_wheel_joint</right_joint>
+            <left_joint>front_left_wheel_joint</left_joint>
+            <right_joint>front_right_wheel_joint</right_joint>
             <!-- Kinematics -->
-            <wheel_separation>0.35</wheel_separation>
-            <wheel_separation>0.35</wheel_separation>
+            <wheel_separation>0.325</wheel_separation>
+            <wheel_separation>0.325</wheel_separation>
             <wheel_diameter>0.1</wheel_diameter>
             <wheel_diameter>0.1</wheel_diameter>

File: description/robot_core.xacro (robot description, xacro)
@@ -1,151 +1,217 @@
 <?xml version="1.0"?>
 <robot xmlns:xacro="http://www.ros.org/wiki/xacro">
-    <!-- SETUP -->
-    <xacro:include filename="inertial_macros.xacro"/>
-    <material name="white">
-        <color rgba="1 1 1 1"/>
-    </material>
-    <material name="orange">
-        <color rgba="1 0.3 0.1 1"/>
-    </material>
-    <material name="blue">
-        <color rgba="0.2 0.2 1 1"/>
-    </material>
-    <material name="black">
-        <color rgba="0 0 0 1"/>
-    </material>
-    <!-- BASE LINK -->
-    <link name="base_link">
+  <!-- Constants for robot dimensions -->
+  <xacro:property name="PI" value="3.1415926535897931"/>
+  <xacro:property name="base_mass" value="4.0" /> <!-- arbitrary value for base mass -->
+  <xacro:property name="base_width" value="0.260" />
+  <xacro:property name="base_length" value="0.525" />
+  <xacro:property name="base_height" value="0.060" />
+  <xacro:property name="wheelbase" value="0.325" />
+  <xacro:property name="wheel_mass" value="0.34055" /> <!-- arbitrary value for wheel mass -->
+  <xacro:property name="wheel_len" value="0.045" />
+  <xacro:property name="wheel_radius" value="0.05" />
+  <!-- <xacro:property name="wheeltrack" value="" -->
+  <!-- Base Link -->
+  <link name="base_link" />
+  <!-- Chassis -->
+  <link name="chassis_link">
+    <collision>
+      <origin xyz="0 0 0" rpy="0 0 0"/>
+      <geometry>
+        <box size="${base_length} ${base_width} ${base_height}"/>
+      </geometry>
+    </collision>
+    <visual>
+      <origin xyz="0 0 0" rpy="0 0 0"/>
+      <geometry>
+        <box size="${base_length} ${base_width} ${base_height}"/>
+      </geometry>
+      <material name="orange"/>
+    </visual>
+    <inertial>
+      <origin xyz="0 0 0" rpy="0 0 0"/>
+      <mass value="${base_mass}"/>
+        <inertia
+          ixx="0.000270" ixy="0.0" ixz="0.0"
+          iyy="0.000270" iyz="0.0"
+          izz="0.000426"/>
+      </inertial>
     </link>
     <joint name="chassis_joint" type="fixed">
-        <parent link="base_link"/>
-        <child link="chassis"/>
-        <origin xyz="-0.1 0 0"/>
-    </joint>
-    <!-- CHASSIS LINK -->
-    <link name="chassis">
+      <parent link="base_link"/>
+      <child link="chassis_link"/>
+      <origin xyz="0 0 ${base_height/2 + wheel_radius}" rpy="0 0 0"/>
+      <axis xyz="0 0 1"/>
+      <dynamics damping="0.2"/>
+    </joint>
+    <!-- rear wheels -->
+    <!-- virtual rear wheel -->
+    <link name="virtual_rear_wheel">
+      <visual>
+        <origin xyz="0 0 0" rpy="${PI/2} 0 ${PI/2}"/>
+        <geometry>
+          <cylinder length="0.01" radius="${wheel_radius}"/>
+        </geometry>
+        <material name="invisible"/>
+      </visual>
+    </link>
+    <joint name="virtual_rear_wheel_joint" type="continuous">
+      <parent link="chassis_link"/>
+      <child link="virtual_rear_wheel"/>
+      <origin xyz="-${wheelbase/2} 0 -${base_height/2}" rpy="0 0 ${PI/2}"/>
+      <axis xyz="1 0 0"/>
+      <limit effort="100.0" velocity="100.0"/>
+      <dynamics damping="0.2"/>
+    </joint>
+    <!-- rear right wheel -->
+    <link name="rear_right_wheel">
+      <collision>
+        <origin xyz="0 0 0" rpy="${PI/2} 0 ${PI/2}"/>
+        <geometry>
+          <cylinder length="${wheel_len}" radius="${wheel_radius}"/>
+        </geometry>
+      </collision>
+      <visual>
+        <origin xyz="0 0 0" rpy="${PI/2} 0 ${PI/2}"/>
+        <geometry>
+          <cylinder length="${wheel_len}" radius="${wheel_radius}"/>
+        </geometry>
+        <material name="black"/>
+      </visual>
+      <inertial>
+        <origin xyz="0 0 0" rpy="${PI/2} 0 ${PI/2}"/>
+        <mass value="${wheel_mass}"/>
+        <inertia
+          ixx="0.000270" ixy="0.0" ixz="0.0"
+          iyy="0.000270" iyz="0.0"
+          izz="0.000426"/>
+      </inertial>
+    </link>
+    <joint name="rear_right_wheel_joint" type="continuous">
+      <parent link="chassis_link"/>
+      <child link="rear_right_wheel"/>
+      <origin xyz="-${wheelbase/2} ${base_width/2} -${base_height/2}" rpy="0 0 ${PI/2}"/>
+      <axis xyz="1 0 0"/>
+      <limit effort="100.0" velocity="100.0"/>
+      <dynamics damping="0.2"/>
+      <mimic joint="virtual_rear_wheel_joint" multiplier="1.0" offset="0.0"/>
+    </joint>
+    <!-- rear left wheel -->
+    <link name="rear_left_wheel">
+        <collision>
+          <origin xyz="0 0 0" rpy="${PI/2} 0 ${PI/2}"/>
+          <geometry>
+            <cylinder length="${wheel_len}" radius="${wheel_radius}"/>
+          </geometry>
+        </collision>
         <visual>
-            <origin xyz="0.25 0 0.075" rpy="0 0 0"/>
-            <geometry>
-                <box size="0.5 0.3 0.15"/>
-            </geometry>
-            <material name="white"/>
+          <origin xyz="0 0 0" rpy="${PI/2} 0 ${PI/2}"/>
+          <geometry>
+            <cylinder length="${wheel_len}" radius="${wheel_radius}"/>
+          </geometry>
+          <material name="black"/>
         </visual>
-        <collision>
-            <origin xyz="0.25 0 0.075" rpy="0 0 0"/>
-            <geometry>
-                <box size="0.5 0.3 0.15"/>
-            </geometry>
-        </collision>
-        <xacro:inertial_box mass="0.5" x="0.5" y="0.3" z="0.15">
-            <origin xyz="0.25 0 0.075" rpy="0 0 0"/>
-        </xacro:inertial_box>
-    </link>
-    <gazebo reference="chassis">
-        <material>Gazebo/White</material>
-    </gazebo>
-    <!-- LEFT FRONT WHEEL -->
-    <joint name="left_front_wheel_joint" type="continuous">
-        <parent link="base_link"/>
-        <child link="left_front_wheel"/>
-        <origin xyz="0.3 0.175 0" rpy="-${pi/2} 0 0"/>
-        <axis xyz="0 0 1"/>
-    </joint>
-    <link name="left_front_wheel">
-        <visual>
-            <geometry>
-                <cylinder length="0.04" radius="0.05" />
-            </geometry>
-            <material name="blue"/>
-        </visual>
-        <collision>
-            <geometry>
-                <cylinder length="0.04" radius="0.05" />
-            </geometry>
-        </collision>
-        <xacro:inertial_cylinder mass="0.1" length="0.04" radius="0.05">
-            <origin xyz="0 0 0" rpy="0 0 0"/>
-        </xacro:inertial_cylinder>
-    </link>
-    <gazebo reference="left_front_wheel">
-        <material>Gazebo/Blue</material>
-    </gazebo>
-    <!-- LEFT REAR WHEEL -->
-    <joint name="left_rear_wheel_joint" type="continuous">
-        <parent link="base_link"/>
-        <child link="left_rear_wheel"/>
-        <origin xyz="0 0.175 0" rpy="-${pi/2} 0 0"/>
-        <axis xyz="0 0 1"/>
-    </joint>
-    <link name="left_rear_wheel">
-        <visual>
-            <geometry>
-                <cylinder length="0.04" radius="0.05" />
-            </geometry>
-            <material name="blue"/>
-        </visual>
-        <collision>
-            <geometry>
-                <cylinder length="0.04" radius="0.05" />
-            </geometry>
-        </collision>
-        <xacro:inertial_cylinder mass="0.1" length="0.04" radius="0.05">
-            <origin xyz="0 0 0" rpy="0 0 0"/>
-        </xacro:inertial_cylinder>
-    </link>
-    <gazebo reference="left_rear_wheel">
-        <material>Gazebo/Blue</material>
-    </gazebo>
-    <!-- RIGHT FRONT WHEEL -->
-    <joint name="right_front_wheel_joint" type="continuous">
-        <parent link="base_link"/>
-        <child link="right_front_wheel"/>
-        <origin xyz="0.3 -0.175 0" rpy="${pi/2} 0 0"/>
-        <axis xyz="0 0 -1"/>
-    </joint>
-    <link name="right_front_wheel">
-        <visual>
-            <geometry>
-                <cylinder length="0.04" radius="0.05" />
-            </geometry>
-            <material name="blue"/>
-        </visual>
-        <collision>
-            <geometry>
-                <cylinder length="0.04" radius="0.05" />
-            </geometry>
-        </collision>
-        <xacro:inertial_cylinder mass="0.1" length="0.04" radius="0.05">
-            <origin xyz="0 0 0" rpy="0 0 0"/>
-        </xacro:inertial_cylinder>
-    </link>
-    <gazebo reference="right_front_wheel">
-        <material>Gazebo/Blue</material>
-    </gazebo>
-    <!-- RIGHT REAR WHEEL -->
-    <joint name="right_rear_wheel_joint" type="continuous">
-        <parent link="base_link"/>
-        <child link="right_rear_wheel"/>
-        <origin xyz="0 -0.175 0" rpy="${pi/2} 0 0"/>
-        <axis xyz="0 0 -1"/>
-    </joint>
-    <link name="right_rear_wheel">
-        <visual>
-            <geometry>
-                <cylinder length="0.04" radius="0.05" />
-            </geometry>
-            <material name="blue"/>
-        </visual>
-        <collision>
-            <geometry>
-                <cylinder length="0.04" radius="0.05" />
-            </geometry>
-        </collision>
-        <xacro:inertial_cylinder mass="0.1" length="0.04" radius="0.05">
-            <origin xyz="0 0 0" rpy="0 0 0"/>
-        </xacro:inertial_cylinder>
-    </link>
-    <gazebo reference="right_rear_wheel">
-        <material>Gazebo/Blue</material>
-    </gazebo>
+        <inertial>
+          <origin xyz="0 0 0" rpy="${PI/2} 0 ${PI/2}"/>
+          <mass value="${wheel_mass}"/>
+          <inertia
+            ixx="0.000270" ixy="0.0" ixz="0.0"
+            iyy="0.000270" iyz="0.0"
+            izz="0.000426"/>
+        </inertial>
+    </link>
+    <joint name="rear_left_wheel_joint" type="continuous">
+      <parent link="chassis_link" />
+      <child link="rear_left_wheel" />
+      <origin xyz="-${wheelbase/2} -${base_width/2} -${base_height/2}" rpy="0 0 ${PI/2}"/>
+      <axis xyz="1 0 0"/>
+      <limit effort="100.0" velocity="100.0"/>
+      <dynamics damping="0.2"/>
+      <mimic joint="virtual_rear_wheel_joint" multiplier="1.0" offset="0.0"/>
+    </joint>
+    <!-- front wheels -->
+    <!-- virtual front wheel -->
+    <link name="virtual_front_wheel">
+      <visual>
+        <origin xyz="0 0 0" rpy="${PI/2} 0 ${PI/2}"/>
+        <geometry>
+          <cylinder length="0.01" radius="${wheel_radius}"/>
+        </geometry>
+        <material name="invisible"/>
+      </visual>
+    </link>
+    <joint name="virtual_front_wheel_joint" type="revolute">
+      <parent link="chassis_link"/>
+      <child link="virtual_front_wheel"/>
+      <origin xyz="${wheelbase/2} 0 -${base_height/2}" rpy="0 0 ${PI/2}"/>
+      <axis xyz="0 0 1"/>
+      <limit lower="-0.4" upper="0.4" effort="100.0" velocity="0.0"/>
+      <dynamics damping="0.2"/>
+    </joint>
+    <!-- front right wheel -->
+    <link name="front_right_wheel">
+      <collision>
+        <origin xyz="0 0 0" rpy="${PI/2} 0 ${PI/2}"/>
+        <geometry>
+          <cylinder length="${wheel_len}" radius="${wheel_radius}"/>
+        </geometry>
+      </collision>
+      <visual>
+        <origin xyz="0 0 0" rpy="${PI/2} 0 ${PI/2}"/>
+        <geometry>
+          <cylinder length="${wheel_len}" radius="${wheel_radius}"/>
+        </geometry>
+        <material name="black"/>
+      </visual>
+      <inertial>
+        <origin xyz="0 0 0" rpy="${PI/2} 0 ${PI/2}"/>
+        <mass value="${wheel_mass}"/>
+        <inertia
+          ixx="0.000270" ixy="0.0" ixz="0.0"
+          iyy="0.000270" iyz="0.0"
+          izz="0.000426"/>
+      </inertial>
+    </link>
+    <joint name="front_right_wheel_joint" type="revolute">
+      <parent link="chassis_link" />
+      <child link="front_right_wheel" />
+      <origin xyz="${wheelbase/2} ${base_width/2} -${base_height/2}" rpy="0 0 ${PI/2}"/>
+      <axis xyz="0 0 1"/>
+      <limit lower="-0.4" upper="0.4" effort="100.0" velocity="0.0"/>
+      <dynamics damping="0.2"/>
+      <mimic joint="virtual_front_wheel_joint" multiplier="1.0" offset="0.0"/>
+    </joint>
+    <!-- front left steering -->
+    <link name="front_left_wheel">
+      <collision>
+        <origin xyz="0 0 0" rpy="${PI/2} 0 ${PI/2}"/>
+        <geometry>
+          <cylinder length="${wheel_len}" radius="${wheel_radius}"/>
+        </geometry>
+      </collision>
+      <visual>
+        <origin xyz="0 0 0" rpy="${PI/2} 0 ${PI/2}"/>
+        <geometry>
+          <cylinder length="${wheel_len}" radius="${wheel_radius}"/>
+        </geometry>
+        <material name="black"/>
+      </visual>
+      <inertial>
+        <origin xyz="0 0 0" rpy="${PI/2} 0 ${PI/2}"/>
+        <mass value="${wheel_mass}"/>
+        <inertia
+          ixx="0.000270" ixy="0.0" ixz="0.0"
+          iyy="0.000270" iyz="0.0"
+          izz="0.000426"/>
+      </inertial>
+    </link>
+    <joint name="front_left_wheel_joint" type="revolute">
+      <parent link="chassis_link" />
+      <child link="front_left_wheel" />
+      <origin xyz="${wheelbase/2} -${base_width/2} -${base_height/2}" rpy="0 0 ${PI/2}"/>
+      <axis xyz="0 0 1"/>
+      <limit lower="-0.4" upper="0.4" effort="100.0" velocity="0.0"/>
+      <dynamics damping="0.2"/>
+      <mimic joint="virtual_front_wheel_joint" multiplier="1.0" offset="0.0"/>
+    </joint>
 </robot>
